Commit message: FR subsystem 완료

File: urdf/crabster_description.urdf (robot description, URDF)
Before this commit: robot crabster, 2 links, 1 joints
Links:
- added link Subsystem11(FR_Yaw_Motor), mass 10.281919; collision mesh filename=package://crabster_simulator/meshes/Subsystem11(FR_Yaw_Moto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; visual mesh filename=package://crabster_simulator/meshes/Subsystem11(FR_Yaw_Moto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
- added link Subsystem12(FR_Roll_Arm), mass 10.085826; collision mesh filename=package://crabster_simulator/meshes/Subsystem12(FR_Roll_Arm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; visual mesh filename=package://crabster_simulator/meshes/Subsystem12(FR_Roll_Arm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
- added link Subsystem13(FR_Pitch_Arm), mass 10.017580; collision mesh filename=package://crabster_simulator/meshes/Subsystem13(FR_Pitch_Ar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; visual mesh filename=package://crabster_simulator/meshes/Subsystem13(FR_Pitch_Ar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
- added link Subsystem14(FR_Leg), mass 20.079610; collision mesh filename=package://crabster_simulator/meshes/Subsystem14(FR_Leg).STL; visual mesh filename=package://crabster_simulator/meshes/Subsystem14(FR_Leg).STL
- added link Subsystem21(MR_Yaw_Motor), mass 10.297182; collision mesh filename=package://crabster_simulator/meshes/Subsystem21(MR_Yaw_Moto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; visual mesh filename=package://crabster_simulator/meshes/Subsystem21(MR_Yaw_Moto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
- added link Subsystem22(MR_Roll_Arm), mass 10.022381; collision mesh filename=package://crabster_simulator/meshes/Subsystem22(MR_Roll_Arm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; visual mesh filename=package://crabster_simulator/meshes/Subsystem22(MR_Roll_Arm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
- added link Subsystem23(MR_Pitch_Arm), mass 10.018527; collision mesh filename=package://crabster_simulator/meshes/Subsystem23(MR_Pitch_Ar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; visual mesh filename=package://crabster_simulator/meshes/Subsystem23(MR_Pitch_Ar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
- added link Subsystem24(MR_Leg), mass 20.080756; collision mesh filename=package://crabster_simulator/meshes/Subsystem24(MR_Leg).STL; visual mesh filename=package://crabster_simulator/meshes/Subsystem24(MR_Leg).STL
- added link Subsystem31(RR_Yaw_Motor), mass 10.297183; collision mesh filename=package://crabster_simulator/meshes/Subsystem31(RR_Yaw_Moto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; visual mesh filename=package://crabster_simulator/meshes/Subsystem31(RR_Yaw_Moto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
- added link Subsystem32(RR_Roll_Arm), mass 10.002542; collision mesh filename=package://crabster_simulator/meshes/Subsystem32(RR_Roll_Arm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; visual mesh filename=package://crabster_simulator/meshes/Subsystem32(RR_Roll_Arm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
- added link Subsystem33(RR_Pitch_Arm), mass 10.018360; collision mesh filename=package://crabster_simulator/meshes/Subsystem33(RR_Pitch_Ar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; visual mesh filename=package://crabster_simulator/meshes/Subsystem33(RR_Pitch_Ar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
- added link Subsystem34(RR_Leg), mass 20.076146; collision mesh filename=package://crabster_simulator/meshes/Subsystem34(RR_Leg).STL; visual mesh filename=package://crabster_simulator/meshes/Subsystem34(RR_Leg).STL
- added link Subsystem41(FL_Yaw_Motor), mass 10.293062; collision mesh filename=package://crabster_simulator/meshes/Subsystem41(FL_Yaw_Moto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; visual mesh filename=package://crabster_simulator/meshes/Subsystem41(FL_Yaw_Moto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
- added link Subsystem42(FL_Roll_Arm), mass 10.035839; collision mesh filename=package://crabster_simulator/meshes/Subsystem42(FL_Roll_Arm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; visual mesh filename=package://crabster_simulator/meshes/Subsystem42(FL_Roll_Arm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
- added link Subsystem43(FL_Pitch_Arm), mass 10.041873; collision mesh filename=package://crabster_simulator/meshes/Subsystem43(FL_Pitch_Ar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; visual mesh filename=package://crabster_simulator/meshes/Subsystem43(FL_Pitch_Ar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
- added link Subsystem44(FL_Leg), mass 20.000655; collision mesh filename=package://crabster_simulator/meshes/Subsystem44(FL_Leg).STL; visual mesh filename=package://crabster_simulator/meshes/Subsystem44(FL_Leg).STL
- added link Subsystem51(ML_Yaw_Motor), mass 10.297596; collision mesh filename=package://crabster_simulator/meshes/Subsystem51(ML_Yaw_Moto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; visual mesh filename=package://crabster_simulator/meshes/Subsystem51(ML_Yaw_Moto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
- added link Subsystem52(ML_Roll_Arm), mass 10.027569; collision mesh filename=package://crabster_simulator/meshes/Subsystem52(ML_Roll_Arm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; visual mesh filename=package://crabster_simulator/meshes/Subsystem52(ML_Roll_Arm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
- added link Subsystem53(ML_Pitch_Arm), mass 10.063326; collision mesh filename=package://crabster_simulator/meshes/Subsystem53(ML_Pitch_Ar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; visual mesh filename=package://crabster_simulator/meshes/Subsystem53(ML_Pitch_Ar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
- added link Subsystem54(ML_Leg), mass 20.065685; collision mesh filename=package://crabster_simulator/meshes/Subsystem54(ML_Leg).STL; visual mesh filename=package://crabster_simulator/meshes/Subsystem54(ML_Leg).STL
- added link Subsystem61(RL_Yaw_Motor), mass 10.297183; collision mesh filename=package://crabster_simulator/meshes/Subsystem61(RL_Yaw_Moto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; visual mesh filename=package://crabster_simulator/meshes/Subsystem61(RL_Yaw_Moto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
- added link Subsystem62(RL_Roll_Arm), mass 10.002542; collision mesh filename=package://crabster_simulator/meshes/Subsystem62(RL_Roll_Arm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; visual mesh filename=package://crabster_simulator/meshes/Subsystem62(RL_Roll_Arm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
- added link Subsystem63(RL_Pitch_Arm), mass 10.042014; collision mesh filename=package://crabster_simulator/meshes/Subsystem63(RL_Pitch_Ar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; visual mesh filename=package://crabster_simulator/meshes/Subsystem63(RL_Pitch_Ar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
- added link Subsystem64(RL_Leg), mass 20.006482; collision mesh filename=package://crabster_simulator/meshes/Subsystem64(RL_Leg).STL; visual mesh filename=package://crabster_simulator/meshes/Subsystem64(RL_Leg).STL
- link BaseBody: mass 100.041 -> 100.040817
Joints:
- added joint BaseBody_to_Subsystem11(FR_Yaw_Motor): type revolute, parent BaseBody, child Subsystem11(FR_Yaw_Motor), origin xyz=0.416200 -0.760100 -0.005500 rpy=0.000000 -0.000000 -0.785398, axis 0 0 1, limit lower=-3.14 upper=3.14 effort=10 velocity=100
- added joint BaseBody_to_Subsystem21(MR_Yaw_Motor): type revolute, parent BaseBody, child Subsystem21(MR_Yaw_Motor), origin xyz=-0.343900 -0.817000 -0.005500 rpy=0.000000 -0.000000 -1.570800, axis 0 0 1, limit lower=-3.14 upper=3.14 effort=10 velocity=100
- added joint BaseBody_to_Subsystem31(RR_Yaw_Motor): type revolute, parent BaseBody, child Subsystem31(RR_Yaw_Motor), origin xyz=-1.102100 -0.748200 -0.005500 rpy=0.000000 -0.000000 -1.745330, axis 0 0 1, limit lower=-3.14 upper=3.14 effort=10 velocity=100
- added joint BaseBody_to_Subsystem41(FL_Yaw_Motor): type revolute, parent BaseBody, child Subsystem41(FL_Yaw_Motor), origin xyz=0.415800 0.760500 -0.005500 rpy=0.000000 -0.000000 0.785398, axis 0 0 1, limit lower=-3.14 upper=3.14 effort=10 velocity=100
- added joint BaseBody_to_Subsystem51(ML_Yaw_Motor): type revolute, parent BaseBody, child Subsystem51(ML_Yaw_Motor), origin xyz=-0.343900 0.817000 -0.005500 rpy=0.000000 -0.000000 1.570800, axis 0 0 1, limit lower=-3.14 upper=3.14 effort=10 velocity=100
- added joint BaseBody_to_Subsystem61(RL_Yaw_Motor): type revolute, parent BaseBody, child Subsystem61(RL_Yaw_Motor), origin xyz=-1.102100 0.748200 -0.005500 rpy=0.000000 -0.000000 1.745330, axis 0 0 1, limit lower=-3.14 upper=3.14 effort=10 velocity=100
- added joint Subsystem11(FR_Yaw_Motor)_to_Subsystem12(FR_Roll_Arm): type revolute, parent Subsystem11(FR_Yaw_Motor), child Subsystem12(FR_Roll_Arm), origin xyz=0.000000 0.000000 0.000000 rpy=-1.570804 -1.047193 0.000009, axis 0 0 1, limit lower=-3.14 upper=3.14 effort=10 velocity=100
- added joint Subsystem12(FR_Roll_Arm)_to_Subsystem13(FR_Pitch_Arm): type revolute, parent Subsystem12(FR_Roll_Arm), child Subsystem13(FR_Pitch_Arm), origin xyz=0.394588 -0.000121 -0.000617 rpy=-2.356194 -1.570791 -0.785394, axis 0 0 1, limit lower=-3.14 upper=3.14 effort=10 velocity=100
- added joint Subsystem13(FR_Pitch_Arm)_to_Subsystem14(FR_Leg): type revolute, parent Subsystem13(FR_Pitch_Arm), child Subsystem14(FR_Leg), origin xyz=-0.000090 0.000026 0.263276 rpy=-1.570800 -0.000003 -1.570793, axis 0 0 1, limit lower=-3.14 upper=3.14 effort=10 velocity=100
- added joint Subsystem21(MR_Yaw_Motor)_to_Subsystem22(MR_Roll_Arm): type revolute, parent Subsystem21(MR_Yaw_Motor), child Subsystem22(MR_Roll_Arm), origin xyz=0.000000 0.000000 0.000000 rpy=-1.570804 -1.047193 0.000004, axis 0 0 1, limit lower=-3.14 upper=3.14 effort=10 velocity=100
- added joint Subsystem22(MR_Roll_Arm)_to_Subsystem23(MR_Pitch_Arm): type revolute, parent Subsystem22(MR_Roll_Arm), child Subsystem23(MR_Pitch_Arm), origin xyz=0.394589 -0.000118 -0.000497 rpy=-2.356194 -1.570791 -0.785394, axis 0 0 1, limit lower=-3.14 upper=3.14 effort=10 velocity=100
- added joint Subsystem23(MR_Pitch_Arm)_to_Subsystem24(MR_Leg): type revolute, parent Subsystem23(MR_Pitch_Arm), child Subsystem24(MR_Leg), origin xyz=-0.000003 -0.000018 0.263185 rpy=-1.570800 -0.000003 -1.570793, axis 0 0 1, limit lower=-3.14 upper=3.14 effort=10 velocity=100
- added joint Subsystem31(RR_Yaw_Motor)_to_Subsystem32(RR_Roll_Arm): type revolute, parent Subsystem31(RR_Yaw_Motor), child Subsystem32(RR_Roll_Arm), origin xyz=0.000000 0.000000 0.000000 rpy=-1.570804 -1.047193 0.000004, axis 0 0 1, limit lower=-3.14 upper=3.14 effort=10 velocity=100
- added joint Subsystem32(RR_Roll_Arm)_to_Subsystem33(RR_Pitch_Arm): type revolute, parent Subsystem32(RR_Roll_Arm), child Subsystem33(RR_Pitch_Arm), origin xyz=0.394592 -0.000114 -0.000510 rpy=0.257951 -1.480877 2.876035, axis 0 0 1, limit lower=-3.14 upper=3.14 effort=10 velocity=100
- added joint Subsystem33(RR_Pitch_Arm)_to_Subsystem34(RR_Leg): type revolute, parent Subsystem33(RR_Pitch_Arm), child Subsystem34(RR_Leg), origin xyz=-0.022817 -0.002213 0.262262 rpy=-1.483858 0.006578 -1.547219, axis 0 0 1, limit lower=-3.14 upper=3.14 effort=10 velocity=100
- added joint Subsystem41(FL_Yaw_Motor)_to_Subsystem42(FL_Roll_Arm): type revolute, parent Subsystem41(FL_Yaw_Motor), child Subsystem42(FL_Roll_Arm), origin xyz=0.000000 0.000000 0.000000 rpy=-1.570804 -1.047193 0.000004, axis 0 0 1, limit lower=-3.14 upper=3.14 effort=10 velocity=100
- added joint Subsystem42(FL_Roll_Arm)_to_Subsystem43(FL_Pitch_Arm): type revolute, parent Subsystem42(FL_Roll_Arm), child Subsystem43(FL_Pitch_Arm), origin xyz=0.394591 -0.000116 0.000057 rpy=-2.356194 -1.570791 -0.785394, axis 0 0 1, limit lower=-3.14 upper=3.14 effort=10 velocity=100
- added joint Subsystem43(FL_Pitch_Arm)_to_Subsystem44(FL_Leg): type revolute, parent Subsystem43(FL_Pitch_Arm), child Subsystem44(FL_Leg), origin xyz=0.000031 0.000031 0.260960 rpy=-1.570800 -0.000003 -1.570793, axis 0 0 1, limit lower=-3.14 upper=3.14 effort=10 velocity=100
- added joint Subsystem51(ML_Yaw_Motor)_to_Subsystem52(ML_Roll_Arm): type revolute, parent Subsystem51(ML_Yaw_Motor), child Subsystem52(ML_Roll_Arm), origin xyz=0.000000 0.000000 0.000000 rpy=-1.570796 -1.047193 -0.000000, axis 0 0 1, limit lower=-3.14 upper=3.14 effort=10 velocity=100
- added joint Subsystem52(ML_Roll_Arm)_to_Subsystem53(ML_Pitch_Arm): type revolute, parent Subsystem52(ML_Roll_Arm), child Subsystem53(ML_Pitch_Arm), origin xyz=0.394594 -0.000111 0.000497 rpy=0.785398 -1.570796 2.356194, axis 0 0 1, limit lower=-3.14 upper=3.14 effort=10 velocity=100
- added joint Subsystem53(ML_Pitch_Arm)_to_Subsystem54(ML_Leg): type revolute, parent Subsystem53(ML_Pitch_Arm), child Subsystem54(ML_Leg), origin xyz=0.000003 -0.000010 0.263181 rpy=-1.570796 -0.000000 -1.570796, axis 0 0 1, limit lower=-3.14 upper=3.14 effort=10 velocity=100
- added joint Subsystem61(RL_Yaw_Motor)_to_Subsystem62(RL_Roll_Arm): type revolute, parent Subsystem61(RL_Yaw_Motor), child Subsystem62(RL_Roll_Arm), origin xyz=0.000000 0.000000 0.000000 rpy=-1.570804 -1.047193 0.000004, axis 0 0 1, limit lower=-3.14 upper=3.14 effort=10 velocity=100
- added joint Subsystem62(RL_Roll_Arm)_to_Subsystem63(RL_Pitch_Arm): type revolute, parent Subsystem62(RL_Roll_Arm), child Subsystem63(RL_Pitch_Arm), origin xyz=0.394596 -0.000106 0.000509 rpy=-2.883555 -1.480878 -0.265645, axis 0 0 1, limit lower=-3.14 upper=3.14 effort=10 velocity=100
- added joint Subsystem63(RL_Pitch_Arm)_to_Subsystem64(RL_Leg): type revolute, parent Subsystem63(RL_Pitch_Arm), child Subsystem64(RL_Leg), origin xyz=0.022901 -0.002308 0.262307 rpy=-1.657732 0.006578 -1.594366, axis 0 0 1, limit lower=-3.14 upper=3.14 effort=10 velocity=100
- joint world_to_BaseBody: origin xyz=0 0 0  rpy=0 0 0 -> xyz=0.000000 0.000000 0.000000 rpy=0.000000 -0.000000 0.000000
