Commit message: full model motion debugging...

File: crabster_visual/urdf/crabster_description.urdf (robot description, URDF)
Before this commit: robot crabster, 26 links, 25 joints
Joints:
- joint BaseBody_to_Subsystem11(FR_Yaw_Motor): limit lower=-3.14 upper=3.14 effort=10 velocity=100 -> lower=-6.28 upper=6.28 effort=100 velocity=100
- joint BaseBody_to_Subsystem21(MR_Yaw_Motor): limit lower=-3.14 upper=3.14 effort=10 velocity=100 -> lower=-6.28 upper=6.28 effort=100 velocity=100
- joint BaseBody_to_Subsystem31(RR_Yaw_Motor): limit lower=-3.14 upper=3.14 effort=10 velocity=100 -> lower=-6.28 upper=6.28 effort=100 velocity=100
- joint BaseBody_to_Subsystem41(FL_Yaw_Motor): limit lower=-3.14 upper=3.14 effort=10 velocity=100 -> lower=-6.28 upper=6.28 effort=100 velocity=100
- joint BaseBody_to_Subsystem51(ML_Yaw_Motor): limit lower=-3.14 upper=3.14 effort=10 velocity=100 -> lower=-6.28 upper=6.28 effort=100 velocity=100
- joint BaseBody_to_Subsystem61(RL_Yaw_Motor): limit lower=-3.14 upper=3.14 effort=10 velocity=100 -> lower=-6.28 upper=6.28 effort=100 velocity=100
- joint Subsystem11(FR_Yaw_Motor)_to_Subsystem12(FR_Roll_Arm): limit lower=-3.14 upper=3.14 effort=10 velocity=100 -> lower=-6.28 upper=6.28 effort=100 velocity=100
- joint Subsystem12(FR_Roll_Arm)_to_Subsystem13(FR_Pitch_Arm): limit lower=-3.14 upper=3.14 effort=10 velocity=100 -> lower=-6.28 upper=6.28 effort=100 velocity=100
- joint Subsystem13(FR_Pitch_Arm)_to_Subsystem14(FR_Leg): limit lower=-3.14 upper=3.14 effort=10 velocity=100 -> lower=-6.28 upper=6.28 effort=100 velocity=100
- joint Subsystem21(MR_Yaw_Motor)_to_Subsystem22(MR_Roll_Arm): limit lower=-3.14 upper=3.14 effort=10 velocity=100 -> lower=-6.28 upper=6.28 effort=100 velocity=100
- joint Subsystem22(MR_Roll_Arm)_to_Subsystem23(MR_Pitch_Arm): limit lower=-3.14 upper=3.14 effort=10 velocity=100 -> lower=-6.28 upper=6.28 effort=100 velocity=100
- joint Subsystem23(MR_Pitch_Arm)_to_Subsystem24(MR_Leg): limit lower=-3.14 upper=3.14 effort=10 velocity=100 -> lower=-6.28 upper=6.28 effort=100 velocity=100
- joint Subsystem31(RR_Yaw_Motor)_to_Subsystem32(RR_Roll_Arm): limit lower=-3.14 upper=3.14 effort=10 velocity=100 -> lower=-6.28 upper=6.28 effort=100 velocity=100
- joint Subsystem32(RR_Roll_Arm)_to_Subsystem33(RR_Pitch_Arm): limit lower=-3.14 upper=3.14 effort=10 velocity=100 -> lower=-6.28 upper=6.28 effort=100 velocity=100
- joint Subsystem33(RR_Pitch_Arm)_to_Subsystem34(RR_Leg): limit lower=-3.14 upper=3.14 effort=10 velocity=100 -> lower=-6.28 upper=6.28 effort=100 velocity=100
- joint Subsystem41(FL_Yaw_Motor)_to_Subsystem42(FL_Roll_Arm): limit lower=-3.14 upper=3.14 effort=10 velocity=100 -> lower=-6.28 upper=6.28 effort=100 velocity=100
- joint Subsystem42(FL_Roll_Arm)_to_Subsystem43(FL_Pitch_Arm): limit lower=-3.14 upper=3.14 effort=10 velocity=100 -> lower=-6.28 upper=6.28 effort=100 velocity=100
- joint Subsystem43(FL_Pitch_Arm)_to_Subsystem44(FL_Leg): limit lower=-3.14 upper=3.14 effort=10 velocity=100 -> lower=-6.28 upper=6.28 effort=100 velocity=100
- joint Subsystem51(ML_Yaw_Motor)_to_Subsystem52(ML_Roll_Arm): limit lower=-3.14 upper=3.14 effort=10 velocity=100 -> lower=-6.28 upper=6.28 effort=100 velocity=100
- joint Subsystem52(ML_Roll_Arm)_to_Subsystem53(ML_Pitch_Arm): limit lower=-3.14 upper=3.14 effort=10 velocity=100 -> lower=-6.28 upper=6.28 effort=100 velocity=100
- joint Subsystem53(ML_Pitch_Arm)_to_Subsystem54(ML_Leg): limit lower=-3.14 upper=3.14 effort=10 velocity=100 -> lower=-6.28 upper=6.28 effort=100 velocity=100
- joint Subsystem61(RL_Yaw_Motor)_to_Subsystem62(RL_Roll_Arm): limit lower=-3.14 upper=3.14 effort=10 velocity=100 -> lower=-6.28 upper=6.28 effort=100 velocity=100
- joint Subsystem62(RL_Roll_Arm)_to_Subsystem63(RL_Pitch_Arm): limit lower=-3.14 upper=3.14 effort=10 velocity=100 -> lower=-6.28 upper=6.28 effort=100 velocity=100
- joint Subsystem63(RL_Pitch_Arm)_to_Subsystem64(RL_Leg): limit lower=-3.14 upper=3.14 effort=10 velocity=100 -> lower=-6.28 upper=6.28 effort=100 velocity=100
